Commit message: feat(vision): mount eye-in-hand RGB-D camera directly on welding arm torch

File: urdf/fixtures/welding_cell_elements.urdf.xacro (robot description, xacro)
@@ -243,54 +243,5 @@
       <child link="clamp_4"/>
     </joint>
-    <!-- 6. OAK-D Lite Depth Camera -->
-    <link name="camera_link">
-      <visual>
-        <origin xyz="0 0 0" rpy="0 0 0"/>
-        <geometry>
-          <mesh filename="package://ventek_autonomous_welding/simulation/cell/meshes/camera_oak_d_lite.dae"/>
-        </geometry>
-        <material name="camera_anodized_black">
-          <color rgba="0.10 0.10 0.12 1.0"/>
-        </material>
-      </visual>
-      <collision>
-        <origin xyz="0 0 0" rpy="0 0 0"/>
-        <geometry>
-          <box size="0.095 0.030 0.030"/>
-        </geometry>
-      </collision>
-      <inertial>
-        <mass value="0.15"/>
-        <origin xyz="0 0 0" rpy="0 0 0"/>
-        <inertia ixx="0.0001" ixy="0" ixz="0" iyy="0.0001" iyz="0" izz="0.0001"/>
-      </inertial>
-    </link>
-    <!-- Camera mounted overlooking workpiece: x=0.85, y=0.0, z=1.35, pitch down 45 deg -->
-    <joint name="camera_joint" type="fixed">
-      <origin xyz="0.85 0.0 1.35" rpy="0 0.785398 3.141592"/>
-      <parent link="${parent}"/>
-      <child link="camera_link"/>
-    </joint>
-    <link name="camera_optical_frame"/>
-    <joint name="camera_optical_joint" type="fixed">
-      <origin xyz="0 0 0" rpy="-1.570796 0 -1.570796"/>
-      <parent link="camera_link"/>
-      <child link="camera_optical_frame"/>
-    </joint>
-    <!-- Alias matching simulation plan (camera_frame) -->
-    <link name="camera_frame"/>
-    <joint name="camera_frame_alias" type="fixed">
-      <origin xyz="0 0 0" rpy="0 0 0"/>
-      <parent link="camera_link"/>
-      <child link="camera_frame"/>
-    </joint>
-    <!-- Alias matching Gazebo Sim frame_id for seamless RViz PointCloud2 & Camera displays -->
-    <link name="oak_d_lite_sensor_model/camera_sensor_link/oak_d_lite_camera"/>
-    <joint name="gz_sensor_frame_joint" type="fixed">
-      <origin xyz="0 0 0" rpy="0 0 0"/>
-      <parent link="camera_link"/>
-      <child link="oak_d_lite_sensor_model/camera_sensor_link/oak_d_lite_camera"/>
-    </joint>
-    <!-- 7. Auxiliary Cell Equipment -->
+    <!-- 6. Auxiliary Cell Equipment -->
     <!-- KUKA KRC4 Robot Controller Cabinet -->
     <link name="krc4_cabinet">
@@ -414,13 +365,4 @@
       </visual>
     </gazebo>
-    <gazebo reference="camera_link">
-      <visual>
-        <material>
-          <ambient>0.06 0.06 0.08 1.0</ambient>
-          <diffuse>0.10 0.10 0.12 1.0</diffuse>
-          <specular>0.20 0.20 0.20 1.0</specular>
-        </material>
-      </visual>
-    </gazebo>
     <gazebo reference="krc4_cabinet">
       <visual>

File: urdf/tool/welding_torch.urdf.xacro (robot description, xacro)
@@ -58,4 +58,97 @@
       <child link="${prefix}tcp_welding_torch"/>
     </joint>
+    <!-- ======================================================================== -->
+    <!-- Eye-in-Hand OAK-D Lite Depth Camera (Mounted on Welding Torch / Arm)     -->
+    <!-- POV directly tracks the welding torch tip and joint seam in real time   -->
+    <!-- ======================================================================== -->
+    <link name="${prefix}camera_link">
+      <visual>
+        <!-- Rotate -90 deg around Z so the 3D model lenses (+Y) point along camera optical axis (+X) -->
+        <origin xyz="0 0 0" rpy="0 0 -1.570796"/>
+        <geometry>
+          <mesh filename="package://ventek_autonomous_welding/simulation/cell/meshes/camera_oak_d_lite.dae"/>
+        </geometry>
+        <material name="camera_anodized_black">
+          <color rgba="0.10 0.10 0.12 1.0"/>
+        </material>
+      </visual>
+      <collision>
+        <origin xyz="0 0 0" rpy="0 0 0"/>
+        <geometry>
+          <box size="0.030 0.095 0.030"/>
+        </geometry>
+      </collision>
+      <inertial>
+        <mass value="0.15"/>
+        <origin xyz="0 0 0" rpy="0 0 0"/>
+        <inertia ixx="0.0001" ixy="0" ixz="0" iyy="0.0001" iyz="0" izz="0.0001"/>
+      </inertial>
+    </link>
+    <!-- Camera mounted on torch bracket: elevated above torch neck, looking at weld seam & nozzle -->
+    <joint name="${prefix}camera_joint" type="fixed">
+      <origin xyz="-0.04 0.0 0.14" rpy="0 0.82 0"/>
+      <parent link="${prefix}welding_torch_link"/>
+      <child link="${prefix}camera_link"/>
+    </joint>
+    <link name="${prefix}camera_optical_frame"/>
+    <joint name="${prefix}camera_optical_joint" type="fixed">
+      <origin xyz="0 0 0" rpy="-1.570796 0 -1.570796"/>
+      <parent link="${prefix}camera_link"/>
+      <child link="${prefix}camera_optical_frame"/>
+    </joint>
+    <!-- Alias matching simulation plan (camera_frame) -->
+    <link name="${prefix}camera_frame"/>
+    <joint name="${prefix}camera_frame_alias" type="fixed">
+      <origin xyz="0 0 0" rpy="0 0 0"/>
+      <parent link="${prefix}camera_link"/>
+      <child link="${prefix}camera_frame"/>
+    </joint>
+    <!-- Alias matching Gazebo Sim frame_ids for seamless RViz PointCloud2 & Camera displays -->
+    <link name="${prefix}oak_d_lite_sensor_model/camera_sensor_link/oak_d_lite_camera"/>
+    <joint name="${prefix}gz_sensor_frame_joint" type="fixed">
+      <origin xyz="0 0 0" rpy="0 0 0"/>
+      <parent link="${prefix}camera_link"/>
+      <child link="${prefix}oak_d_lite_sensor_model/camera_sensor_link/oak_d_lite_camera"/>
+    </joint>
+    <link name="${prefix}ventek_welding_cell/camera_link/oak_d_lite_camera"/>
+    <joint name="${prefix}gz_sensor_cell_frame_joint" type="fixed">
+      <origin xyz="0 0 0" rpy="0 0 0"/>
+      <parent link="${prefix}camera_link"/>
+      <child link="${prefix}ventek_welding_cell/camera_link/oak_d_lite_camera"/>
+    </joint>
+    <!-- Gazebo Shading & Moving Eye-in-Hand RGB-D Camera Sensor -->
+    <gazebo reference="${prefix}camera_link">
+      <visual>
+        <material>
+          <ambient>0.06 0.06 0.08 1.0</ambient>
+          <diffuse>0.10 0.10 0.12 1.0</diffuse>
+          <specular>0.20 0.20 0.20 1.0</specular>
+        </material>
+      </visual>
+      <sensor name="oak_d_lite_camera" type="rgbd_camera">
+        <camera>
+          <horizontal_fov>1.204</horizontal_fov>
+          <image>
+            <width>640</width>
+            <height>480</height>
+            <format>R8G8B8</format>
+          </image>
+          <clip>
+            <near>0.05</near>
+            <far>4.0</far>
+          </clip>
+          <depth_camera>
+            <clip>
+              <near>0.05</near>
+              <far>4.0</far>
+            </clip>
+          </depth_camera>
+        </camera>
+        <always_on>true</always_on>
+        <update_rate>30</update_rate>
+        <visualize>true</visualize>
+        <topic>/ventek/vision/camera</topic>
+      </sensor>
+    </gazebo>
   </xacro:macro>
 </robot>

File: urdf/welding_cell/welding_cell.urdf (robot description, URDF)
Before this commit: robot ventek_welding_cell, 29 links, 28 joints
Links:
- added link oak_d_lite_sensor_model/camera_sensor_link/oak_d_lite_camera
- added link ventek_welding_cell/camera_link/oak_d_lite_camera
- link camera_link: geometry collision box size=0.030 0.095 0.030; visual mesh filename=package://ventek_autonomous_welding/simulation/cell/meshes/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
Joints:
- added joint gz_sensor_cell_frame_joint: type fixed, parent camera_link, child ventek_welding_cell/camera_link/oak_d_lite_camera, origin xyz=0 0 0 rpy=0 0 0
- added joint gz_sensor_frame_joint: type fixed, parent camera_link, child oak_d_lite_sensor_model/camera_sensor_link/oak_d_lite_camera, origin xyz=0 0 0 rpy=0 0 0
- joint camera_joint: origin xyz=0.85 0.0 1.35 rpy=0 0.785398 3.141592 -> xyz=-0.04 0.0 0.14 rpy=0 0.82 0; parent world -> welding_torch_link
